File: sensor_python300/sensor_python300.kicad_sch (KiCad schematic)
At the start: 78 parts, among them J101 DF40HC(4.0)-60DS-0.4V(51), U101 NOIP1SN0300A-QTI, U102 TPS7A2033PDBVR, U103 TPS22918DBVR, U104 TPS7A2033PDBVR, U105 APX803S-29SA-7, U106 TPS610995DRVR, X101 <DNP> DSC1103DI5-360.0000

Commit message: KiCAD 10.0 へ
Parts:
- TP103, TP104, TP105, TP106, TP107, TP108, TP109: value ~ -> (none)
